File: PCB/CE-PiicoDev-Buzzer.kicad_sch (KiCad schematic)
At the start: 23 parts, among them SW1 ADDR, U1 ATtiny806

Commit message: V20 (#1)
* provisional v20 design

* v20
Parts:
- removed J2: (no value), symbol CoreElectronics_Components:Conn_PiicoDev_socket_UPDI
- removed JP3, JP5: SolderJumper_2_Open, Jumper:SolderJumper-2_P1.3mm_Open_RoundedPad1.0x1.5mm, symbol Jumper:SolderJumper_2_Open
- removed LS1: Speaker_Crystal, Buzzer_Beeper:Buzzer_Murata_PKMCS0909E, symbol Device:Speaker_Crystal
- removed SW1: ADDR, CoreElectronics_Components:SW_DIP_SPSTx02_Slide_DSHP, symbol Switch:SW_DIP_x02
- added C2: 10u, Capacitor_SMD:C_0603_1608Metric, symbol Device:C
- added D2: SS14, Diode_SMD:D_SMA, symbol Device:D_Schottky
- added J2: (no value), CoreElectronics_Components:JST_SH_SM04B-SRSS-TB_1x04-1MP_P1.00mm_Horizontal, symbol Connector:Conn_01x04_Male
- added J3: Conn_01x05_Male, CoreElectronics_Components:TestPoint_Pad_D1.0mm_x05_Pattern1, symbol Connector:Conn_01x05_Male
- added J4: RX, TestPoint:TestPoint_Pad_D1.5mm, symbol Connector:Conn_01x01_Male
- added J5: TX, TestPoint:TestPoint_Pad_D1.5mm, symbol Connector:Conn_01x01_Male
- added LS1: MLT-8540H, Buzzer:CUI_CMT-8540S-SMT, symbol Device:Speaker
- added Q1: BSS138, Package_TO_SOT_SMD:SOT-23, symbol Transistor_FET:BSS138
- added R6: 10k, Resistor_SMD:R_0402_1005Metric, symbol Device:R
- added SW1: ID, CoreElectronics_Components:SW_DIP_x04_Slide_CHS-04A1, symbol Switch:SW_DIP_x04
- FID1, FID2: value (none) -> Fiducial; footprint (none) -> CoreElectronics_Components:Fiducial_1mm_Mask2mm_No_Courtyard
- H1, H2: value (none) -> MountingHole; footprint (none) -> CoreElectronics_Components:MountingHole_2.7mm_M2.5_PadClearance_1.2
- J1: value (none) -> (none); footprint (none) -> CoreElectronics_Components:JST_SH_SM04B-SRSS-TB_1x04-1MP_P1.00mm_Horizontal
- JP2: value (none) -> I2C PU; footprint (none) -> CoreElectronics_Components:SolderJumper-3_P1.3mm_Closed_RoundedPad1.0x1.5mm_NumberLabels; symbol PiicoDev-Buzzer-rescue:SolderJumper_3_Bridged123-Jumper -> Jumper:SolderJumper_3_Bridged123
- R2, R3: value (none) -> 10k; footprint (none) -> Resistor_SMD:R_0402_1005Metric
- R4, R5: value (none) -> 120R; footprint (none) -> Resistor_SMD:R_0402_1005Metric
- U1: value ATtiny806 -> ATtiny1616-M
Connections:
- net +3V3: now also R5.2, J2.2 (Pin_2), J3.2 (Pin_2)
- net ADD1: now also U1.7 (PA6), SW1.1; no longer U1.8 (PA7)
- net ADD2: now also U1.8 (PA7), SW1.2; no longer U1.9 (PB5)
- net ADD3: now also U1.9 (PB5), SW1.3; no longer U1.6 (PA5)
- net ADD4: now also U1.10 (PB4), SW1.4; no longer U1.12 (PB2)
- net GND: now also C2.2, J2.1 (Pin_1), J3.1 (Pin_1), Q1.2 (S), SW1.5, SW1.6, SW1.7, SW1.8
- net PWR_LED: now also U1.2 (PA3); no longer U1.17 (PC2)
- net SCL: now also J2.4 (Pin_4), J3.4 (Pin_4)
- net SDA: now also R4.2, J2.3 (Pin_3), J3.3 (Pin_3); no longer U1.13 (PB1)
- net UPDI: now also J3.5 (Pin_5)
- net UART_RX: now reaches U1.11 (PB3)
- net UART_RX: now also J4.1 (Pin_1)
- net BUZZ: no longer names the net of U1.5 (PA4)
- net BUZZ_1: no longer names the net of R4.1
- net BUZZ_1: now also U1.13 (PB1); no longer U1.2 (PA3)
- net BUZZ_2: no longer names the net of U1.20 (PA1)
- net BUZZ_2: no longer R5.1
- removed net BUZZ_3: R4.2, R5.2, U1.1 (PA2)
- new net: Q1.1 (G), R6.2
- new net: D2.2 (A), LS1.2, Q1.3 (D)
- new net: C2.1, D2.1 (K), LS1.1, R5.1
- new net BUZZER: R6.1, U1.1 (PA2)
- new net UART_TX: J5.1 (Pin_1), U1.12 (PB2)
- no-connect marks 0 -> 7
Other:
- note added: "Programming and Test"
- title: PiicoDev Buzzer Module -> PiicoDev Buzzer
- moved on the sheet: C1, U1
